File: Placa_Madre/sensores.kicad_sch (KiCad schematic)
At the start: 5 parts, among them J1 Conn_01x10_Pin, J2 Conn_01x10_Pin, U1 MCP3008, U2 MCP3008

Commit message: Add files via upload
Parts:
- removed J1, J2: Conn_01x10_Pin, symbol Connector:Conn_01x10_Pin
- added J3, J4: Conn_01x20_Pin, Connector_PinHeader_1.00mm:PinHeader_1x20_P1.00mm_Vertical, symbol Connector:Conn_01x20_Pin
- added R16, R17, R18, R19, R20, R21, R22, R23, R24, R25, R26, R27, R28, R29, R30, R31: R, Resistor_SMD:R_0201_0603Metric, symbol Device:R
- RP1: footprint RASPBERRYPI -> imprtdasd:MODULE_RASPBERRY_PI_4B_4GB
- U1, U2: footprint (none) -> imprtdasd:DIP16-2.54-19.2X7.62MM
Connections:
- net at RP1.1 (+3.3V_1): now also U1.15 (Vref), U1.16 (Vdd)
- net at RP1.14 (GND_3): now also U1.14 (AGND), U1.9 (DGND), J3.10 (Pin_10), J3.11 (Pin_11), J3.12 (Pin_12), J3.13 (Pin_13), J3.14 (Pin_14), J3.15 (Pin_15), J3.16 (Pin_16), J3.17 (Pin_17), J3.18 (Pin_18), J3.9 (Pin_9)
- net at RP1.17 (+3.3V_2): now also U2.15 (Vref), U2.16 (Vdd)
- net at RP1.19 (GPIO_10/SPI0_MOSI): now also U1.11 (Din)
- net at RP1.21 (GPIO_9/SPI0_MISO): now also U1.12 (Dout)
- net at RP1.23 (GPIO_11/SPI0_SCLK): now also U1.13 (CLK)
- net at RP1.24 (GPIO_8/SPI0_CE1_N): now also U1.10 (~{CS}/SHDN)
- net at RP1.25 (GND_5): now also U2.14 (AGND), U2.9 (DGND), J4.10 (Pin_10), J4.11 (Pin_11), J4.12 (Pin_12), J4.6 (Pin_6), J4.7 (Pin_7), J4.8 (Pin_8), J4.9 (Pin_9)
- net at RP1.26 (GPIO_7/SPI0_CE2_N): now also U2.10 (~{CS}/SHDN)
- net at RP1.35 (GPIO19/SPI0_MISO1/PWM1): now also U2.12 (Dout)
- net at RP1.38 (GPIO20/SPI0_MOSI1): now also U2.11 (Din)
- net at RP1.40 (GPIO21/SPI0_SCLK1): now also U2.13 (CLK)
- net at U2.1 (CH0): now also R31.1
- net at U2.2 (CH1): now also R30.1
- net at U2.3 (CH2): now also R29.1
- net at U2.4 (CH3): now also R28.1
- net at U2.5 (CH4): now also R27.1
- net at U2.6 (CH5): now also R26.1
- net at U2.7 (CH6): now also R25.1
- net at U2.8 (CH7): now also R24.1
- net at U1.1 (CH0): now also R23.2
- net at U1.2 (CH1): now also R22.2
- net at U1.3 (CH2): now also R21.2
- net at U1.4 (CH3): now also R20.2
- net at U1.5 (CH4): now also R19.2
- net at U1.6 (CH5): now also R18.2
- net at U1.7 (CH6): now also R17.2
- net at U1.8 (CH7): now also R16.2
- new net: J3.1 (Pin_1), R23.1
- new net: J3.2 (Pin_2), R22.1
- new net: J3.3 (Pin_3), R21.1
- new net: J3.4 (Pin_4), R20.1
- new net: J3.5 (Pin_5), R19.1
- new net: J3.6 (Pin_6), R18.1
- new net: J3.7 (Pin_7), R17.1
- new net: J3.8 (Pin_8), R16.1
- new net: J4.18 (Pin_18), R26.2
- new net: J4.14 (Pin_14), R30.2
- new net: J4.13 (Pin_13), R31.2
- new net: J4.15 (Pin_15), R29.2
- new net: J4.16 (Pin_16), R28.2
- new net: J4.17 (Pin_17), R27.2
- new net: J4.19 (Pin_19), R25.2
- new net: J4.20 (Pin_20), R24.2
Other:
- moved on the sheet: RP1, U1, U2
