File: Placa_Madre/sensores.kicad_sch (KiCad schematic)
At the start: 21 parts, among them J1 Raspberry_Pi_4, J3 Conn_01x20_Pin, J4 Conn_01x20_Pin, U1 MCP3008, U2 MCP3008

Commit message: Add files via upload
Connections:
- net 18 is gone; now on net GND: J3.10 (Pin_10), J3.11 (Pin_11), J3.12 (Pin_12), J3.13 (Pin_13), J3.14 (Pin_14), J3.15 (Pin_15), J3.16 (Pin_16), J3.17 (Pin_17), J3.18 (Pin_18), J3.9 (Pin_9)
- net GND: now also U1.14 (AGND), U1.9 (DGND)
