File: Placa_Madre/sensores.kicad_pcb (KiCad board)
At the start: 2 copper layers, 21 parts, among them J3 Conn_01x20_Pin, J4 Conn_01x20_Pin, U1 MCP3008, U2 MCP3008

Commit message: Add files via upload
Parts:
- moved R19 47.1 mm to (141.8, 103.6), turned to 180 degrees
- moved R17 47.0 mm to (141.8, 107.1), turned to 180 degrees
- moved R18 46.9 mm to (141.8, 105.3), turned to 180 degrees
- moved R23 42.2 mm to (139.3, 103.6), turned to 180 degrees
- moved R21 42.1 mm to (139.3, 107.1), turned to 180 degrees
- moved R22 42.0 mm to (139.3, 105.3), turned to 180 degrees
- moved R27 37.3 mm to (136.8, 103.6), turned to 180 degrees
- moved R25 37.2 mm to (136.8, 107.1), turned to 180 degrees
- moved R26 37.1 mm to (136.8, 105.3), turned to 180 degrees
- moved R31 32.5 mm to (134.4, 103.6), turned to 180 degrees
- moved R29 32.3 mm to (134.4, 107.1), turned to 180 degrees
- moved R30 32.2 mm to (134.4, 105.3), turned to 180 degrees
- moved J4 25.8 mm to (50.7, 119.5), turned to 180 degrees
- moved J3 21.0 mm to (54.0, 119.5), turned to 180 degrees
- moved R28 15.7 mm to (87.1, 107.1), turned to -90 degrees
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