File: Placa_Madre/sensor.kicad_sch (KiCad schematic)
At the start: 10 parts, among them J1 Screw_Terminal_01x02, J2 Screw_Terminal_01x04, J3 Screw_Terminal_01x04, J4 Screw_Terminal_01x04, J5 Screw_Terminal_01x02, J6 Screw_Terminal_01x02, U1 RASPBERRY_PI_4B_4GB, U2 TMC2208_SILENTSTEPSTICK, U3 TMC2208_SILENTSTEPSTICK, U4 TMC2208_SILENTSTEPSTICK

Commit message: Add files via upload
Parts:
- removed J2, J3, J4: Screw_Terminal_01x04, TerminalBlock_Phoenix:TerminalBlock_Phoenix_MPT-0,5-4-2.54_1x04_P2.54mm_Horizontal, symbol Connector:Screw_Terminal_01x04
- added J2, J3, J4, J7, J8, J9: Screw_Terminal_01x02, TerminalBlock_MetzConnect:TerminalBlock_MetzConnect_360272_1x01_Horizontal_ScrewM2.6, symbol Connector:Screw_Terminal_01x02
- J1, J5, J6: footprint TerminalBlock_Phoenix:TerminalBlock_Phoenix_MPT-0,5-2-2.54_1x02_P2.54mm_Horizontal -> TerminalBlock_MetzConnect:TerminalBlock_MetzConnect_360272_1x01_Horizontal_ScrewM2.6
Connections:
- net at U4.JP2_4 (OA1): now also J8.1 (Pin_1)
- net at U4.JP2_3 (OA2): now also J8.2 (Pin_2)
- net at U4.JP2_5 (OB1): now also J9.1 (Pin_1)
- net at U4.JP2_6 (OB2): now also J9.2 (Pin_2)
- net at U2.JP2_4 (OA1): now also J7.1 (Pin_1)
- net at U2.JP2_3 (OA2): now also J7.2 (Pin_2)
- net at U2.JP2_5 (OB1): now also J4.1 (Pin_1)
- net at U2.JP2_6 (OB2): now also J4.2 (Pin_2)
- net at U3.JP2_4 (OA1): now also J3.1 (Pin_1)
- net at U3.JP2_3 (OA2): now also J3.2 (Pin_2)
- net at U3.JP2_5 (OB1): now also J2.1 (Pin_1)
- net at U3.JP2_6 (OB2): now also J2.2 (Pin_2)

Commit message: update
Parts:
- removed U1: RASPBERRY_PI_4B_4GB, pi 4:MODULE_RASPBERRY_PI_4B_4GB, symbol Pi 4:RASPBERRY_PI_4B_4GB
- added J10: Screw_Terminal_01x02, TerminalBlock_MetzConnect:TerminalBlock_MetzConnect_360272_1x01_Horizontal_ScrewM2.6, symbol Connector:Screw_Terminal_01x02
- added U1: RASPBERRY_PI_PICO, pi pico:RASPBERRY_PI_PICO, symbol pi pico:RASPBERRY_PI_PICO
Connections:
- net VIO2 is gone; now on net VIO: U4.JP2_7 (VIO)
- net DIR: now also U1.GND3
- net DIR2: now also U1.GP19
- net DIR3: now also U1.GP21
- net GND: now also U1.GND
- net STEP1: now also U1.GP18
- net STEP2: now also U1.GP20
- net STEP3: now also U1.GP22
- net VIO: now also U1.3V3
- new net: J10.2 (Pin_2), U1.GP0
- new net: J10.1 (Pin_1), U1.GP1
